Commit message: Minor logging and arg updates, fix panda_wristcam initial pose

File: mani_skill/assets/robots/panda/panda_v3.urdf (robot description, URDF)
Before this commit: robot panda, 15 links, 14 joints
Joints:
- joint panda_hand_joint: origin xyz=0 0 0 rpy=0 0 -0.7853981633974483 -> xyz=0 0 0 rpy=0 0 0.7853981633974483
