Commit message: Update reachy_mobile

File: mani_skill/assets/robots/reachy/reachy_mobile.urdf (robot description, URDF)
Before this commit: robot reachy_2023, 39 links, 38 joints
Links:
- link base_link: mass 20 -> 24.0; geometry collision cylinder length=0.2609 radius=0.245; visual mesh filename=zuuu_description/meshes/mobile_base_visual.dae
