Commit message: Add base mobility, fix collisions, revert gripper to original mimics with updated limits

File: mani_skill/assets/robots/reachy/reachy2_mod.urdf (robot description, URDF)
Before this commit: robot reachy2, 96 links, 95 joints
Links:
- added link root, mass 0
- added link root_arm_1_link_1, mass 0
- added link root_arm_1_link_2, mass 0
Joints:
- added joint root_x_axis_joint: type prismatic, parent root, child root_arm_1_link_1, axis 1 0 0, limit lower=-20 upper=20 effort=100 velocity=0.50
- added joint root_y_axis_joint: type prismatic, parent root_arm_1_link_1, child root_arm_1_link_2, axis 0 1 0, limit lower=-20 upper=20 effort=100 velocity=0.50
- added joint root_z_rotation_joint: type continuous, parent root_arm_1_link_2, child base_link, axis 0 0 1
- joint l_hand_finger: limit lower=0.0 upper=2.27 effort=100.0 velocity=10.0 -> lower=0.3 upper=0.75 effort=100.0 velocity=10.0
- joint l_hand_finger_distal: mimic (none) -> joint=l_hand_finger multiplier=0.4689 offset=-0.554
- joint l_hand_finger_distal_mimic: mimic joint=l_hand_finger_distal multiplier=1 offset=0 -> joint=l_hand_finger multiplier=0.4689 offset=-0.554
- joint l_hand_finger_proximal: mimic (none) -> joint=l_hand_finger multiplier=-0.4689 offset=0.554
- joint r_hand_finger: limit lower=0.0 upper=2.27 effort=100.0 velocity=10.0 -> lower=0.3 upper=0.75 effort=100.0 velocity=10.0
- joint r_hand_finger_distal: mimic (none) -> joint=r_hand_finger multiplier=0.4689 offset=-0.554
- joint r_hand_finger_distal_mimic: mimic joint=r_hand_finger_distal multiplier=1 offset=0 -> joint=r_hand_finger multiplier=0.4689 offset=-0.554
- joint r_hand_finger_proximal: mimic (none) -> joint=r_hand_finger multiplier=-0.4689 offset=0.554

Commit message: Fix tripod anchors, update keyframe qposes

File: mani_skill/assets/robots/reachy/reachy2_mod.urdf (robot description, URDF)
Before this commit: robot reachy2, 99 links, 98 joints
Links:
- link left_bar_anchor: geometry collision box size=0.03 0.03 0.005; visual box size=0.03 0.03 0.005
- link left_bar_base: geometry collision box size=0.01 0.05 0.485; collision box size=0.01 0.05 0.485
- link right_bar_anchor: geometry collision box size=0.03 0.03 0.005; visual box size=0.03 0.03 0.005
- link right_bar_base: geometry collision box size=0.01 0.05 0.485; collision box size=0.01 0.05 0.485
