Commit message: Update reachy2_static for PickCube

File: mani_skill/assets/robots/reachy/reachy2_static.urdf (robot description, URDF)
Before this commit: robot reachy_static, 30 links, 29 joints
Links:
- link bottom_neck_arm: geometry collision cylinder length=0.0 radius=0.0; visual mesh filename=reachy_description/meshes_old/orbita_arm.dae
- link head: geometry collision cylinder length=0.15 radius=0.06; visual mesh filename=reachy_description/meshes_old/head.dae
- link l_antenna_link: geometry collision cylinder length=0.0 radius=0.0; visual mesh filename=reachy_description/meshes_old/antenna.dae
- link l_forearm: geometry collision cylinder length=0.09 radius=0.04; visual mesh filename=reachy_description/meshes_old/forearm.dae
- link l_gripper_finger: geometry collision box size=0.05 0.012 0.035; visual mesh filename=reachy_description/meshes_old/l_gripper_finger.dae
- link l_gripper_thumb: geometry collision box size=0.1 0.012 0.035; visual mesh filename=reachy_description/meshes_old/l_gripper_thumb.dae
- link l_shoulder: geometry collision cylinder length=0.09 radius=0.035; visual mesh filename=reachy_description/meshes_old/shoulder.dae
- link l_shoulder_x: geometry collision cylinder length=0.04 radius=0.035; visual mesh filename=reachy_description/meshes_old/shoulder_x.dae
- link l_upper_arm: geometry collision cylinder length=0.25 radius=0.04; visual mesh filename=reachy_description/meshes_old/upper_arm.dae
- link l_wrist: geometry collision cylinder length=0.14 radius=0.035; visual mesh filename=reachy_description/meshes_old/wrist.dae
- link l_wrist2hand: geometry collision cylinder length=0.03 radius=0.025; visual mesh filename=reachy_description/meshes_old/wrist2hand.dae
- link middle_neck_arm: geometry collision cylinder length=0.0 radius=0.0; visual mesh filename=reachy_description/meshes_old/orbita_arm.dae
- link r_antenna_link: geometry collision cylinder length=0.0 radius=0.0; visual mesh filename=reachy_description/meshes_old/antenna.dae
- link r_forearm: geometry collision cylinder length=0.09 radius=0.04; visual mesh filename=reachy_description/meshes_old/forearm.dae
- link r_gripper_finger: geometry collision box size=0.05 0.012 0.035; visual mesh filename=reachy_description/meshes_old/r_gripper_finger.dae
- link r_gripper_thumb: geometry collision box size=0.1 0.012 0.035; visual mesh filename=reachy_description/meshes_old/r_gripper_thumb.dae
- link r_shoulder: geometry collision cylinder length=0.09 radius=0.035; visual mesh filename=reachy_description/meshes_old/shoulder.dae
- link r_shoulder_x: geometry collision cylinder length=0.04 radius=0.035; visual mesh filename=reachy_description/meshes_old/shoulder_x.dae
- link r_upper_arm: geometry collision cylinder length=0.25 radius=0.04; visual mesh filename=reachy_description/meshes_old/upper_arm.dae
- link r_wrist: geometry collision cylinder length=0.14 radius=0.035; visual mesh filename=reachy_description/meshes_old/wrist.dae
- link r_wrist2hand: geometry collision cylinder length=0.03 radius=0.025; visual mesh filename=reachy_description/meshes_old/wrist2hand.dae
- link top_neck_arm: geometry collision cylinder length=0.0 radius=0.0; visual mesh filename=reachy_description/meshes_old/orbita_arm.dae
- link torso: geometry collision box size=0.11 0.2 0.32; visual mesh filename=reachy_description/meshes_old/torso.dae
Joints:
- joint l_gripper: limit lower=-0.35 upper=1.2 effort=10. velocity=0.0 -> lower=0.175 upper=1.2 effort=10. velocity=0.0
- joint r_gripper: limit lower=-1.2 upper=0.35 effort=10. velocity=0.0 -> lower=-0.35 upper=0.8 effort=10. velocity=0.0
